File: midi10trigger.brd (EAGLE design)
At the start: 100 x 80 mm, 42 parts, among them IC1 ATMega328p, IC2 78L05, Q1 20MHz, U1 THONKICONNNEW, U10 THONKICONNNEW, U11 THONKICONNNEW, U12 THONKICONNNEW, U13 THONKICONNNEW, U2 THONKICONNNEW, U3 THONKICONNNEW, U4 THONKICONNNEW, U5 THONKICONNNEW, U6 THONKICONNNEW, U7 THONKICONNNEW, U8 THONKICONNNEW, U9 THONKICONNNEW

Commit message: Add files via upload
reworked
Parts:
- removed MIDI_IN, MIDI_OUT: (no value), og-midi:MAB5SH
- removed SV1: EURO_POWER_HEADERREGULAR, MusicThingModular:EURO_POWER_HEADER
- removed SW7: (no value), og-switch:B3F-40XX
- added D3: 1N4148DO35-7, diode:DO35-7
- added LED10, LED11, LED12, LED13, LED3, LED4, LED5, LED6, LED7, LED8, LED9: TLLG4400, led:LED3MM
- added PAD1: midi in pin 4, wirepad:2,54/1,1
- added PAD2: midi in pin 5, wirepad:2,54/1,1
- added R10, R11, R12, R13, R14, R15, R16, R17, R18, R9: 10K, MusicThingModular:VERTICAL_RESISTOR
- added SV7: EURO_POWER_HEADERFAT_PADS, MusicThingModular:EURO_PWR_HEADER_FAT
- added U$1: SUBMINI_SPDT, MusicThingModular:SUBMINI_TOGGLE
- L1: device rcl:0207/10 -> MusicThingModular:VERTICAL_RESISTOR
- R1, R2, R4, R5, R6, R7, R8: device rcl:0204/7 -> MusicThingModular:VERTICAL_RESISTOR
- R3: value 220 -> 10K; device rcl:0204/7 -> MusicThingModular:VERTICAL_RESISTOR
- moved U11 215.7 mm to (30.9, 63.9), turned to 270 degrees
- moved U13 209.9 mm to (4.83, 62.5)
- moved U12 209.8 mm to (14.9, 62.5)
- moved U10 209.7 mm to (30.9, 74.0), turned to 270 degrees
- moved U9 204.4 mm to (30.9, 84.2), turned to 270 degrees
- moved U8 200.1 mm to (30.9, 94.4), turned to 270 degrees
- moved U7 196.7 mm to (30.9, 104.5), turned to 270 degrees
- moved U6 194.3 mm to (30.9, 114.7), turned to 270 degrees
- moved U5 142.9 mm to (6.86, 74.0), turned to 90 degrees
- moved U1 142.5 mm to (6.86, 114.7), turned to 90 degrees
- moved U4 140.7 mm to (6.86, 84.2), turned to 90 degrees
- moved U2 140.5 mm to (6.86, 104.5), turned to 90 degrees
- moved U3 139.8 mm to (6.86, 94.4), turned to 90 degrees
- moved R7 99.2 mm to (30.2, 30.5)
- moved L1 98.7 mm to (35.4, 23.6), turned to 270 degrees
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Connections:
- removed net START_STOP_OUT: IC1.25, U11.P$1_TIP
- removed net TIG10_OUT: IC1.28
- new net +12: D3.A, SV7.10, SV7.9
- new net -12: SV7.1, SV7.2
- new net N$17: LED3.A, R9.2
- new net N$18: LED4.A, R10.2
- new net N$19: LED5.A, R11.2
- new net N$20: LED6.A, R12.2
- new net N$21: LED7.A, R13.2
- new net N$22: LED8.A, R14.2
- new net N$23: LED9.A, R15.2
- new net N$24: LED10.A, R16.2
- new net N$25: LED11.A, R17.2
- new net N$26: LED12.A, R18.2
- new net TRIG11_OUT: IC1.25, R3.1, U11.P$1_TIP
- net GND: now also LED10.K, LED11.K, LED12.K, LED13.K, LED3.K, LED4.K, LED5.K, LED6.K, LED7.K, LED8.K, LED9.K, SV7.3, SV7.4, SV7.5, SV7.6, SV7.7, SV7.8, U$1.3; no longer MIDI_OUT.2, SW7.1, SW7.2
- net MIDI_OUT: no longer MIDI_OUT.5
- net MISO: now also U$1.1, U$1.COM; no longer SW7.3, SW7.4
- net N$3: now also LED13.A, R3.2; no longer MIDI_OUT.4, R3.1
- net N$72: now also PAD1.1; no longer MIDI_IN.4
- net N$73: now also PAD2.1; no longer MIDI_IN.5
- net TRIG10_OUT: now also IC1.28, R18.1
- net TRIG1_OUT: now also R9.1
- net TRIG2_OUT: now also R10.1
- net TRIG3_OUT: now also R11.1
- net TRIG4_OUT: now also R12.1
- net TRIG5_OUT: now also R13.1
- net TRIG6_OUT: now also R14.1
- net TRIG7_OUT: now also R15.1
- net TRIG8_OUT: now also R16.1
- net TRIG9_OUT: now also R17.1
- net VCC: no longer R3.2
- net VDD: now also D3.C
Routing:
- net GND: track 0.00 -> 283.8 mm, vias 0 -> 4
- net VCC: track 0.00 -> 149.8 mm, vias 0 -> 3
- net TRIG6_OUT: track 0.00 -> 99.9 mm, vias 0 -> 2
- net TRIG7_OUT: track 0.00 -> 88.5 mm, vias 0 -> 1
- net TRIG1_OUT: track 0.00 -> 83.8 mm, vias 0 -> 1
- net TRIG8_OUT: track 0.00 -> 75.6 mm
- net TRIG2_OUT: track 0.00 -> 69.5 mm, vias 0 -> 3
- net TRIG9_OUT: track 0.00 -> 63.4 mm, vias 0 -> 1
- net MISO: track 0.00 -> 60.0 mm, vias 0 -> 1
- net TRIG3_OUT: track 0.00 -> 59.9 mm, vias 0 -> 2
- net N$4: track 0.00 -> 59.1 mm, vias 0 -> 4
- net MOSI: track 0.00 -> 53.6 mm, vias 0 -> 3
- net TRIG4_OUT: track 0.00 -> 52.5 mm, vias 0 -> 2
- net CLOCK_OUT: track 0.00 -> 51.9 mm, vias 0 -> 2
- net SCK: track 0.00 -> 50.7 mm, vias 0 -> 1
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- added copper zone on layer 1, net GND
- added copper zone on layer 16, net GND
Other:
- board size 100 x 80 mm -> 37.8 x 100.3 mm
