File: midi10trigger.sch (EAGLE design)
At the start: 42 parts, among them IC1 ATMega328p, IC2 78L05, Q1 20MHz, U1 THONKICONNNEW, U10 THONKICONNNEW, U11 THONKICONNNEW, U12 THONKICONNNEW, U13 THONKICONNNEW, U2 THONKICONNNEW, U3 THONKICONNNEW, U4 THONKICONNNEW, U5 THONKICONNNEW, U6 THONKICONNNEW, U7 THONKICONNNEW, U8 THONKICONNNEW, U9 THONKICONNNEW

Commit message: Add files via upload
reworked
Parts:
- removed MIDI_IN, MIDI_OUT: MAB5SH, og-midi:MAB5SH
- removed SV1: EURO_POWER_HEADERREGULAR, MusicThingModular:EURO_POWER_HEADERREGULAR
- removed SW7: (no value), og-switch:40-XX
- added D3: 1N4148DO35-7, diode:1N4148DO35-7
- added LED10, LED11, LED12, LED13, LED3, LED4, LED5, LED6, LED7, LED8, LED9: TLLG4400, led:TLLG4400
- added PAD1: midi in pin 4, wirepad:2,54/1,1
- added PAD2: midi in pin 5, wirepad:2,54/1,1
- added R10, R11, R12, R13, R14, R15, R16, R17, R18, R9: 10K, MusicThingModular:RESISTORVERTICAL
- added SV7: EURO_POWER_HEADERFAT_PADS, MusicThingModular:EURO_POWER_HEADERFAT_PADS
- added U$1: SUBMINI_SPDT, MusicThingModular:SUBMINI_SPDT
- L1: device rcl:L-US0207/10 -> MusicThingModular:RESISTORVERTICAL
- R1, R2, R4, R5, R6, R7, R8: device rcl:R-US_0204/7 -> MusicThingModular:RESISTORVERTICAL
- R3: value 220 -> 10K; device rcl:R-US_0204/7 -> MusicThingModular:RESISTORVERTICAL
Connections:
- removed net START_STOP_OUT: IC1.PC2(ADC2), U11.TIP
- removed net TIG10_OUT: IC1.PC5(ADC5/SCL)
- new net +12: D3.A, SV7.10, SV7.9
- new net -12: SV7.1, SV7.2
- new net N$17: LED3.A, R9.2
- new net N$18: LED4.A, R10.2
- new net N$19: LED5.A, R11.2
- new net N$20: LED6.A, R12.2
- new net N$21: LED7.A, R13.2
- new net N$22: LED8.A, R14.2
- new net N$23: LED9.A, R15.2
- new net N$24: LED10.A, R16.2
- new net N$25: LED11.A, R17.2
- new net N$26: LED12.A, R18.2
- new net TRIG11_OUT: IC1.PC2(ADC2), R3.1, U11.TIP
- net GND: now also LED10.C, LED11.C, LED12.C, LED13.C, LED3.C, LED4.C, LED5.C, LED6.C, LED7.C, LED8.C, LED9.C, SV7.3, SV7.4, SV7.5, SV7.6, SV7.7, SV7.8, U$1.S; no longer MIDI_OUT.2, SW7.S, SW7.S1
- net MIDI_OUT: no longer MIDI_OUT.5
- net MISO: now also U$1.COMMON, U$1.O; no longer SW7.P, SW7.P1
- net N$3: now also LED13.A, R3.2; no longer MIDI_OUT.4, R3.1
- net N$72: now also PAD1.P; no longer MIDI_IN.4
- net N$73: now also PAD2.P; no longer MIDI_IN.5
- net TRIG10_OUT: now also IC1.PC5(ADC5/SCL), R18.1
- net TRIG1_OUT: now also R9.1
- net TRIG2_OUT: now also R10.1
- net TRIG3_OUT: now also R11.1
- net TRIG4_OUT: now also R12.1
- net TRIG5_OUT: now also R13.1
- net TRIG6_OUT: now also R14.1
- net TRIG7_OUT: now also R15.1
- net TRIG8_OUT: now also R16.1
- net TRIG9_OUT: now also R17.1
- net VCC: no longer R3.2
- net VDD: now also D3.C
Other:
- moved on the sheet: C5, C6, C7, D1, D2, IC2, ISP, LED1, LED2, OK1, U1, U10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
